Commit message: Use the amber bottle and its PP25 cap in the uncap-and-pipette hand
The MuJoCo scene, the URDFs, the .blend and the viewer now take the 60 ml
amber bottle of assets/amber-bottles with its PP25 cap instead of the iris
clamp kit's placeholder bottle. Its Ø28 mm ribbed cap is the one the clamp
was built for; the blades close on its Ø28.8 mm tamper band (74.8 deg).
Masses come from the meshes (57.8 g, 2.5 g), the thread is PP25 (2.75 mm
pitch, 5.5 mm rise, hinge follows 3.5 deg), and the bottle still collides
as a hollow ring of boxes so the pipette goes down the neck. All MuJoCo
checks pass.

FULL_PHYSICS_ISAAC.md is rewritten from the current MuJoCo state: the
baseline to match, collision filtering the URDF cannot carry (the clamp
envelopes and the cap's solid cylinder would fight the pose writes), contact
scale, and staged pass criteria for grip, blades and thread.

Co-Authored-By: Claude Opus 5 <noreply@anthropic.com>
Claude-Session: https://claude.ai/code/session_01C2eAFRL9sfLHdEAcabR3zt

File: simulation/assets/ur10e_iris_pipette/reference_bottle.urdf (robot description, URDF)
Before this commit: robot reference_bottle, 1 links, 0 joints
Links:
- link reference_bottle: mass 0.12 -> 0.0577634; geometry collision box size=0.002 0.00716085 0.06325; collision box size=0.002 0.00716085 0.06325

File: simulation/assets/ur10e_iris_pipette/reference_cap.urdf (robot description, URDF)
Before this commit: robot reference_cap, 1 links, 0 joints
Links:
- link reference_cap: mass 0.012 -> 0.00246002; geometry collision cylinder length=0.0185 radius=0.0144; visual mesh filename=meshes/amber_cap.stl

File: simulation/models/iris_pipette_rig.urdf (robot description, URDF)
Before this commit: robot iris_pipette_rig, 36 links, 35 joints
Links:
- link hand_frame: mass 0.19451 -> 0.192439; geometry visual box size=0.008 0.006 0.01; visual box size=0.008 0.006 0.01
Joints:
- joint clamp_swing: origin xyz=-0.09 0 0.0815 rpy=0 0 0 -> xyz=-0.09 0 0.0796 rpy=0 0 0
- joint hand_frame_mount: origin xyz=-3.46945e-18 -0.046 0.151038 rpy=-1.5708 -1.5708 0 -> xyz=0 -0.0441 0.152926 rpy=-1.5708 -1.5708 0
- joint hand_mount: origin xyz=-0.151038 0 0.046 rpy=1.5708 0 1.5708 -> xyz=-0.152926 0 0.0441 rpy=1.5708 0 1.5708
- joint pipette_slide: origin xyz=0 0 0.113 rpy=0 0 0 -> xyz=0 0 0.11 rpy=0 0 0
