Commit message: Rebuild the vertical hand assets for the narrow cage page
gripper-design/vertical_hand.html is now the 154 mm U-channel cage: the iris
clamp slides back along X on the +Y plate (parked at x = -90 under the
pipette), the micropipette hangs fixed on the bottle's axis and only goes
down, the jaws reach their carriages through tabs in their own comb bands,
21 steps. vertical_hand_rig.py mirrors the page's new parameter block, state
and joint tree (19 joints, 8 actuated, no swing); the generator builds the
windowed side plates, the back plate, the servo head, the X rail and the
fixed pipette, and its checks and the MuJoCo playback are retargeted to the
new step numbers. All four outputs still agree with fk within 0.03 um and
the sequence passes in MuJoCo.

Co-Authored-By: Claude Fable 5.1 <noreply@anthropic.com>

File: simulation/assets/vertical_hand/vertical_hand.urdf (robot description, URDF)
Before this commit: robot vertical_hand, 21 links, 20 joints
Links:
- removed link pip_swing
- link pip_slide: mass 0.25 -> 0.4; geometry collision cylinder length=0.09 radius=0.0058; visual mesh filename=meshes/pip_slide__blue.stl
Joints:
- removed joint clamp_y
- removed joint pip_swing
- added joint clamp_x: type prismatic, parent hand, child clamp_slide, origin xyz=0 0 0 rpy=0 0 0, axis 1 0 0, limit lower=-0.1 upper=0 effort=200 velocity=2.0
- joint pip_slide: limit lower=0.01 upper=0.15 effort=200 velocity=2.0 -> lower=0.01 upper=0.25 effort=200 velocity=2.0
- joint plunger: origin xyz=-0.03 0.09 0 rpy=0 0 0 -> xyz=0 0 0 rpy=0 0 0; parent pip_swing -> pip_slide

Commit message: Vertical hand: no arm stub, collision on every part, approach and retreat
The model now ends at the servo head's top plate; the UR flange and arm stub
are gone. Every mesh builder carries a collision spec, so the MJCF and the
URDF get a physical body for each part: boxes for the softened boxes and the
cradles (chord boxes along the parabola, liner plus plate), cylinders for the
turned parts, rings as circles of boxes with open bores, the side plates as
two slabs plus a convex hull for the toe. 322 primitives; hand parts collide
with the bottle, the cap and the floor, never with each other. The URDF's
collision geoms are checked against the MJCF's in MuJoCo.

A new `approach` joint (property hand_x) slides the whole hand along X: the
sequence starts 120 mm behind the bottle, advances onto its axis, runs the
page's 21 steps and backs away at the end (23 steps, 32.5 s). The playback
checks the hand returns where it started, and passes with the contacts live.

Co-Authored-By: Claude Fable 5.1 <noreply@anthropic.com>

File: simulation/assets/vertical_hand/vertical_hand.urdf (robot description, URDF)
Before this commit: robot vertical_hand, 20 links, 19 joints
Links:
- added link approach, mass 0.5
- link blade_0: geometry collision box size=0.012 0.062 0.0025; collision cylinder length=0.0025 radius=0.006
- link blade_1: geometry collision box size=0.012 0.062 0.0025; collision cylinder length=0.0025 radius=0.006
- link blade_2: geometry collision box size=0.012 0.062 0.0025; collision cylinder length=0.0025 radius=0.006
- link blade_3: geometry collision box size=0.012 0.062 0.0025; collision cylinder length=0.0025 radius=0.006
- link blade_4: geometry collision box size=0.012 0.062 0.0025; collision cylinder length=0.0025 radius=0.006
- link blade_5: geometry collision box size=0.012 0.062 0.0025; collision cylinder length=0.0025 radius=0.006
- link cam: geometry collision box size=0.005 0.0122437 0.003; collision box size=0.005 0.0122437 0.003
- link clamp_lift: geometry collision box size=0.022 0.032 0.038; collision box size=0.024 0.06 0.008
- link clamp_slide: geometry collision box size=0.014 0.024 0.0724; collision box size=0.04 0.033 0.03
- link hand: geometry collision box size=0.004 0.146 0.4849; collision box size=0.006 0.146 0.016
- link housing: geometry collision box size=0.01 0.014 0.042; collision box size=0.01 0.014 0.042
- link jaw_l: geometry collision box size=0.00412311 0.00925 0.032; collision box size=0.00412311 0.00925 0.032
- link jaw_r: geometry collision box size=0.00412311 0.00925 0.032; collision box size=0.00412311 0.00925 0.032
- link pip_slide: geometry collision box size=0.0045 0.00586791 0.016; collision box size=0.0045 0.00586791 0.016
- link planet_0: geometry collision cylinder length=0.008 radius=0.012; visual mesh filename=meshes/planet_0__housing.stl
- link planet_1: geometry collision cylinder length=0.008 radius=0.012; visual mesh filename=meshes/planet_1__housing.stl
- link planet_2: geometry collision cylinder length=0.008 radius=0.012; visual mesh filename=meshes/planet_2__housing.stl
- link plunger: geometry collision cylinder length=0.0085 radius=0.0085; collision cylinder length=0.026 radius=0.003
- link sun: geometry collision cylinder length=0.008 radius=0.012; collision cylinder length=0.04 radius=0.004
Joints:
- added joint approach: type prismatic, parent vertical_hand, child approach, origin xyz=0 0 0 rpy=0 0 0, axis 1 0 0, limit lower=-0.2 upper=0.05 effort=200 velocity=2.0
- joint lift: parent vertical_hand -> approach
